File: kicad/8_bit_computer/register.kicad_sch (KiCad schematic)
At the start: 26 parts, among them U7 74LS245, U8 74LS173, U9 74LS173

Commit message: Add pull up/down resistors to all vcc/gnd shorts
Parts:
- added R34, R35, R36: 10K, Resistor_THT:R_Axial_DIN0207_L6.3mm_D2.5mm_P7.62mm_Horizontal, symbol Device:R
Connections:
- net +5V: now also R34.1; no longer U7.1 (A->B)
- net GND: now also R35.2, R36.2; no longer U8.1 (Oe1), U8.2 (Oe2), U9.1 (Oe1), U9.2 (Oe2)
- new net: R34.2, U7.1 (A->B)
- new net: R36.1, U9.1 (Oe1), U9.2 (Oe2)
- new net: R35.1, U8.1 (Oe1), U8.2 (Oe2)
